Commit message: Re-posicionamiento de IMU en AIRI.
Signed-off-by: Michel Hidalgo <hid.michel@gmail.com>

File: airi_description/urdf/airi.urdf.xacro (robot description, xacro)
@@ -30,9 +30,9 @@
   <xacro:gy521-imu name="imu"/>
   <xacro:fastener on="base" bears="imu">
-    <origin xyz="0 0 0"/>
+    <origin xyz="0 0 ${board_support_z_offset}"/>
   </xacro:fastener>
   <xacro:rplidar-a1m8r1 name="laser"/>
   <xacro:fastener on="base" bears="laser">
-    <origin xyz="0 0 0.067"/>
+    <origin xyz="0 0 ${board_support_z_offset}"/>
   </xacro:fastener>
   <xacro:ky033-ranger name="left_cliff_sensor"/>

File: airi_description/urdf/parts.urdf.xacro (robot description, xacro)
@@ -2,4 +2,5 @@
 <robot name="parts" xmlns:xacro="http://www.ros.org/wiki/xacro">
   <xacro:property name="wheel_base" value="0.242"/>
+  <xacro:property name="board_support_z_offset" value="0.067"/>
   <xacro:property name="sonar_elevation_angle" value="${-15.0 * PI / 180.0}"/>
   <xacro:property name="sonar_r_offset" value="${0.004 * cos(-sonar_elevation_angle) + 0.170}"/>

Commit message: Contactos espurios en bumper eliminados.
Signed-off-by: Michel Hidalgo <hid.michel@gmail.com>

File: airi_description/urdf/airi.urdf.xacro (robot description, xacro)
@@ -32,5 +32,5 @@
     <origin xyz="0 0 ${board_support_z_offset}"/>
   </xacro:fastener>
-  <xacro:rplidar-a1m8r1 name="laser"/>
+  <xacro:rplidar-a1m8r1 name="laser" topic="scan"/>
   <xacro:fastener on="base" bears="laser">
     <origin xyz="0 0 ${board_support_z_offset}"/>

File: airi_description/urdf/parts.urdf.xacro (robot description, xacro)
@@ -86,5 +86,5 @@
         </material>
       </visual>
-      <selfCollide>true</selfCollide>
+      <self_collide>1</self_collide>
     </gazebo>
     <link name="${name}_bay">
@@ -107,5 +107,5 @@
         </material>
       </visual>
-      <selfCollide>true</selfCollide>
+      <self_collide>1</self_collide>
     </gazebo>
     <joint name="${name}_bay_fastener" type="fixed">
@@ -147,5 +147,5 @@
         </material>
       </visual>
-      <selfCollide>true</selfCollide>
+      <self_collide>1</self_collide>
     </gazebo>
     <joint name="${name}_cover_fastener" type="fixed">
@@ -203,5 +203,5 @@
           <contact>
             <ode>
-              <kp>1.0e6</kp>
+              <kp>1.0e8</kp>
               <kd>1.0</kd>
               <max_vel>0.0</max_vel>
@@ -254,4 +254,5 @@
         </material>
       </visual>
+      <self_collide>1</self_collide>
     </gazebo>
     <link name="${name}_ball">
@@ -292,8 +293,8 @@
           <contact>
             <ode>
-              <kp>1.0e6</kp>
+              <kp>1.0e8</kp>
               <kd>1.0</kd>
               <max_vel>0.0</max_vel>
-              <min_depth>0.0005</min_depth>
+              <min_depth>0.0</min_depth>
             </ode>
           </contact>
@@ -301,4 +302,5 @@
         <max_contacts>1</max_contacts>
       </collision>
+      <self_collide>1</self_collide>
     </gazebo>
     <joint name="${name}_ball_holder" type="fixed">
@@ -331,17 +333,8 @@
     </gazebo>
     <link name="${name}_ball">
-      <inertial>
-        <mass value="${ball_mass}"/>
-        <xacro:sphere_inertia mass="${ball_mass}" radius="${ball_radius}"/>
-      </inertial>
-      <collision>
+       <visual>
         <geometry>
           <sphere radius="${ball_radius}"/>
         </geometry>
-      </collision>
-      <visual>
-        <geometry>
-          <sphere radius="${ball_radius}"/>
-        </geometry>
         <material name="steel"/>
       </visual>
@@ -356,24 +349,4 @@
         </material>
       </visual>
-      <collision>
-        <surface>
-          <friction>
-            <ode>
-              <mu>0.001</mu>
-              <mu2>0.001</mu2>
-              <fdir1>1 0 0</fdir1>
-            </ode>
-          </friction>
-          <contact>
-            <ode>
-              <kp>1.0e6</kp>
-              <kd>1.0</kd>
-              <max_vel>0.0</max_vel>
-              <min_depth>0.0005</min_depth>
-            </ode>
-          </contact>
-        </surface>
-        <max_contacts>1</max_contacts>
-      </collision>
     </gazebo>
     <joint name="${name}_ball_holder" type="fixed">
@@ -395,19 +368,5 @@
                  izz="0.0016116796150935037"/>
       </inertial>
-      <collision name="left_patch">
-        <origin xyz="0 0 ${-bumper_height/2 - bumper_z_offset}"/>
-        <geometry>
-          <mesh filename="package://airi_description/media/parts/left_bumper_patch.stl"
-                scale="0.001 0.001 0.001"/>
-        </geometry>
-      </collision>
-      <collision name="right_patch">
-        <origin xyz="0 0 ${-bumper_height/2 - bumper_z_offset}"/>
-        <geometry>
-          <mesh filename="package://airi_description/media/parts/right_bumper_patch.stl"
-                scale="0.001 0.001 0.001"/>
-        </geometry>
-      </collision>
-      <visual>
+      <collision name="main">
         <origin xyz="0 0 ${-bumper_height/2 - bumper_z_offset - chassis_z_offset}"/>
         <geometry>
@@ -415,4 +374,11 @@
                 scale="0.001 0.001 0.001"/>
         </geometry>
+      </collision>
+      <visual>
+        <origin xyz="0 0 ${-bumper_height/2 - bumper_z_offset - chassis_z_offset}"/>
+        <geometry>
+          <mesh filename="package://airi_description/media/parts/bumper.stl"
+                scale="0.001 0.001 0.001"/>
+        </geometry>
         <material name="thermoplastic"/>
       </visual>
@@ -427,5 +393,5 @@
         </material>
       </visual>
-      <self_collide>true</self_collide>
+      <self_collide>1</self_collide>
       <sensor type="contact" name="${name}">
         <pose>0 0 0 0 0 0</pose>
@@ -433,7 +399,6 @@
         <update_rate>10</update_rate>
         <contact>
-          <!-- Use collision names as it results from URDF to SDF conversion-->
-          <collision>bumper_link_fixed_joint_lump__left_patch_collision</collision>
-          <collision>bumper_link_fixed_joint_lump__right_patch_collision_1</collision>
+          <!-- Use collision names as it results from URDF to SDF conversion -->
+          <collision>bumper_link_fixed_joint_lump__main_collision</collision>
         </contact>
         <plugin name="${name}_controller" filename="libairi_bumper_plugin.so">
@@ -467,4 +432,7 @@
       </visual>
     </link>
+    <gazebo reference="${name}_link">
+      <self_collide>1</self_collide>
+    </gazebo>
   </xacro:macro>
 </robot>

File: airi_description/urdf/sensors.urdf.xacro (robot description, xacro)
@@ -4,5 +4,5 @@
   <xacro:property name="rplidar_a1m8r1_diameter" value="0.070"/>
   <xacro:property name="rplidar_a1m8r1_length" value="0.0245"/>
-  <xacro:macro name="rplidar-a1m8r1" params="name">
+  <xacro:macro name="rplidar-a1m8r1" params="name topic">
     <link name="${name}_link">
       <inertial>
@@ -56,8 +56,9 @@
         </ray>
         <plugin name="${name}_controller" filename="libgazebo_ros_laser.so">
-          <topicName>${name}</topicName>
+          <topicName>${topic}</topicName>
           <frameName>${name}_optical_link</frameName>
         </plugin>
       </sensor>
+      <self_collide>1</self_collide>
     </gazebo>
   </xacro:macro>
@@ -119,4 +120,5 @@
         </plugin>
       </sensor>
+      <self_collide>1</self_collide>
     </gazebo>
   </xacro:macro>
@@ -178,4 +180,5 @@
         </plugin>
       </sensor>
+      <self_collide>1</self_collide>
     </gazebo>
   </xacro:macro>
@@ -213,4 +216,5 @@
         </plugin>
       </sensor>
+      <self_collide>1</self_collide>
     </gazebo>
   </xacro:macro>
