Commit message: Modify vel threshold among other changes.

File: airi_description/urdf/sensors.urdf.xacro (robot description, xacro)
@@ -24,5 +24,5 @@
       <parent link="${name}_link"/>
       <child link="${name}_optical_link"/>
-      <origin xyz="0 0 0.045"/>
+      <origin xyz="0 0 0.045" rpy="0 0 3.141592653589793"/>
     </joint>
     <gazebo reference="${name}_optical_link">
